File: sheet/Lichtwecker/Lichtwecker.kicad_sch (KiCad schematic)
At the start: 1 part

Commit message: OPT: Schaltplan angepasst
Parts:
- added C1: 1000uF, Capacitor_SMD:CP_Elec_6.3x5.9, symbol Device:C_Polarized
- added J1: Conn_01x04_Pin, Connector_Harwin:Harwin_M20-89004xx_1x04_P2.54mm_Horizontal, symbol Connector:Conn_01x04_Pin
- added R1: 470k, Resistor_THT:R_Axial_DIN0204_L3.6mm_D1.6mm_P1.90mm_Vertical, symbol Device:R
- added U1, U2: adafruit-MAX98357, adafruit-MAX98357:adafruit-MAX98357, symbol adafruit-MAX98357:adafruit-MAX98357
- added U3: ~, 01_MyLib:3.5_TFT_Touch_SPI_Display, symbol my_Library:3.5_TFT_Touch_SPI_Display
Connections:
- net +5V: now also C1.1, J1.1 (Pin_1), R1.1, U1.1 (Vin), U1.3 (~{SD_MODE}), U2.1 (Vin), U3.1 (SD_CS)
- net GND: now also C1.2, J1.4 (Pin_4), U1.2 (GND), U2.2 (GND), U3.2 (SD_MOSI)
- net at MOD1.11 (IO_34): now also U3.12 (TP_DIN), U3.6 (TFT_SDI)
- net at MOD1.14 (IO_05/D8): now also U3.3 (SD_MISO)
- net at MOD1.18 (IO_13/TCK): now also U3.5 (TFT_DC_RS)
- net at MOD1.20 (IO_10/SD3): now also U3.11 (TP_CS)
- net at MOD1.24 (IO_27): now also U1.6 (BCLK), U2.6 (BCLK)
- net at MOD1.25 (IO_22/D1/SCL): now also U3.8 (LED)
- net at MOD1.26 (IO_25): now also U1.5 (DIN), U2.5 (DIN)
- net at MOD1.27 (IO_21/D2/SDA): now also U3.14 (TP_IRQ)
- net at MOD1.29 (IO_17/D3): now also U3.4 (SD_CLK)
- net RGB_SDA: now reaches MOD1.37 (TD0)
- net RGB_SDA: now also J1.2 (Pin_2)
- net at MOD1.6 (IO_26/D0): now also U1.7 (LRC), U2.7 (LRC)
- net at MOD1.8 (IO_18/D5): now also U3.10 (TP_CLK), U3.7 (TFT_SCK)
- net at MOD1.9 (IO_33): now also U3.13 (TP_OUT)
- new net: R1.2, U2.3 (~{SD_MODE})
- new net GRÜN: J1.3 (Pin_3)
Other:
- note added: "+5V vom USB"
